Commit message: Added jt_cartesian_controller

File: lwr_description/model/kuka_lwr.gazebo.xacro (robot description, xacro)
@@ -2,8 +2,13 @@
 <robot xmlns:xacro="http://ros.org/wiki/xacro">
 	<xacro:macro name="kuka_lwr_gazebo" params="name">
+<!--
 		<gazebo>
 			<plugin name="gazebo_ros_control" filename="libgazebo_ros_control.so">
 				<robotNamespace>${name}</robotNamespace>
 			</plugin>
+		</gazebo>
+-->
+		<gazebo>
+			<plugin name="ros_control" filename="libgazebo_ros_control.so"/>
 		</gazebo>
 		<gazebo reference="${name}_base_link">

File: lwr_description/model/kuka_lwr.transmission.xacro (robot description, xacro)
@@ -1,75 +1,26 @@
 <?xml version="1.0"?>
 <robot xmlns:xacro="http://ros.org/wiki/xacro">
+  <!-- Transmission Macro -->
+  <xacro:macro name="simple_transmission" params="name joint">
+	<transmission name="${name}_${joint}_trans" type="transmission_interface/SimpleTransmission">
+		<type>transmission_interface/SimpleTransmission</type>
+		<joint name="${name}_${joint}_joint">
+			<hardwareInterface>EffortJointInterface</hardwareInterface>
+		</joint>
+		<actuator name="${name}_${joint}_motor">
+			<hardwareInterface>EffortJointInterface</hardwareInterface>
+			<mechanicalReduction>1</mechanicalReduction>
+		</actuator>
+		<mechanicalReduction>1</mechanicalReduction>
+	</transmission>
+  </xacro:macro>
     <xacro:macro name="kuka_lwr_transmission" params="name">
-	    <transmission name="${name}_0_trans">
-			<type>transmission_interface/SimpleTransmission</type>
-			<joint name="${name}_0_joint">
-				<hardwareInterface>EffortJointInterface</hardwareInterface>
-			</joint>
-			<actuator name="${name}_0_motor">
-				<hardwareInterface>EffortJointInterface</hardwareInterface>
-				<mechanicalReduction>1</mechanicalReduction>
-			</actuator>
-	    </transmission>
-		<transmission name="${name}_1_trans">
-			<type>transmission_interface/SimpleTransmission</type>
-			<joint name="${name}_1_joint">
-				<hardwareInterface>EffortJointInterface</hardwareInterface>
-			</joint>
-			<actuator name="${name}_1_motor">
-				<hardwareInterface>EffortJointInterface</hardwareInterface>
-				<mechanicalReduction>1</mechanicalReduction>
-			</actuator>
-		</transmission>
-		<transmission name="${name}_2_trans">
-			<type>transmission_interface/SimpleTransmission</type>
-			<joint name="${name}_2_joint">
-				<hardwareInterface>EffortJointInterface</hardwareInterface>
-			</joint>
-			<actuator name="${name}_2_motor">
-				<hardwareInterface>EffortJointInterface</hardwareInterface>
-				<mechanicalReduction>1</mechanicalReduction>
-			</actuator>
-		</transmission>
-		<transmission name="${name}_3_trans">
-			<type>transmission_interface/SimpleTransmission</type>
-			<joint name="${name}_3_joint">
-				<hardwareInterface>EffortJointInterface</hardwareInterface>
-			</joint>
-			<actuator name="${name}_3_motor">
-				<hardwareInterface>EffortJointInterface</hardwareInterface>
-				<mechanicalReduction>1</mechanicalReduction>
-			</actuator>
-		</transmission>
-		<transmission name="${name}_4_trans">
-			<type>transmission_interface/SimpleTransmission</type>
-			<joint name="${name}_4_joint">
-				<hardwareInterface>EffortJointInterface</hardwareInterface>
-			</joint>
-			<actuator name="${name}_4_motor">
-				<hardwareInterface>EffortJointInterface</hardwareInterface>
-				<mechanicalReduction>1</mechanicalReduction>
-			</actuator>
-		</transmission>
-		<transmission name="${name}_5_trans">
-			<type>transmission_interface/SimpleTransmission</type>
-			<joint name="${name}_5_joint">
-				<hardwareInterface>EffortJointInterface</hardwareInterface>
-			</joint>
-			<actuator name="${name}_5_motor">
-				<hardwareInterface>EffortJointInterface</hardwareInterface>
-				<mechanicalReduction>1</mechanicalReduction>
-			</actuator>
-		</transmission>
-		<transmission name="${name}_6_trans">
-			<type>transmission_interface/SimpleTransmission</type>
-			<joint name="${name}_6_joint">
-				<hardwareInterface>EffortJointInterface</hardwareInterface>
-			</joint>
-			<actuator name="${name}_6_motor">
-				<hardwareInterface>EffortJointInterface</hardwareInterface>
-				<mechanicalReduction>1</mechanicalReduction>
-			</actuator>
-		</transmission>
+		<simple_transmission name ="${name}" joint="0" />
+		<simple_transmission name ="${name}" joint="1" />
+		<simple_transmission name ="${name}" joint="2" />
+		<simple_transmission name ="${name}" joint="3" />
+		<simple_transmission name ="${name}" joint="4" />
+		<simple_transmission name ="${name}" joint="5" />
+		<simple_transmission name ="${name}" joint="6" />
 	</xacro:macro>
 </robot>

File: lwr_description/model/kuka_lwr.urdf.xacro (robot description, xacro)
@@ -47,5 +47,7 @@
 		<axis xyz="0 0 1"/>
 		<limit lower="${-170 * M_PI / 180}" upper="${170 * M_PI / 180}" effort="204" velocity="${velocity_scale * 110 * M_PI / 180}" />
+<!--
 		<safety_controller soft_lower_limit="${-168 * M_PI / 180}" soft_upper_limit="${168 * M_PI / 180}" k_position="30" k_velocity="30"/>
+-->
 		<dynamics friction="10.0" damping="1.0"/>
 		<parent link="${name}_base_link"/>
@@ -91,5 +93,7 @@
 		<limit lower="${-120 * M_PI / 180}" upper="${120 * M_PI / 180}"
 			 effort="306" velocity="${velocity_scale * 110 * M_PI / 180}" />
+<!--
 		<safety_controller soft_lower_limit="${-118 * M_PI / 180}" soft_upper_limit="${118 * M_PI / 180}" k_position="30" k_velocity="30"/>
+-->
 		<dynamics friction="10.0" damping="1.0"/>
 		<parent link="${name}_1_link"/>
@@ -134,5 +138,7 @@
 		<axis xyz="0 0 1"/>
 		<limit lower="${-170 * M_PI / 180}" upper="${170 * M_PI / 180}" effort="204" velocity="${velocity_scale * 130 * M_PI / 180}" />
+<!--
 		<safety_controller soft_lower_limit="${-168 * M_PI / 180}" soft_upper_limit="${168 * M_PI / 180}" k_position="30" k_velocity="30"/>
+-->
 		<dynamics friction="10.0" damping="1.0"/>
 		<parent link="${name}_2_link"/>
@@ -177,5 +183,7 @@
 		<axis xyz="0 1 0"/>
 		<limit lower="${-120 * M_PI / 180}" upper="${120 * M_PI / 180}" effort="306" velocity="${velocity_scale * 130 * M_PI / 180}" />
+<!--
 			<safety_controller soft_lower_limit="${-118 * M_PI / 180}" soft_upper_limit="${118 * M_PI / 180}" k_position="30" k_velocity="30"/>
+-->
 		<dynamics friction="10.0" damping="1.0"/>
 		<parent link="${name}_3_link"/>
@@ -220,5 +228,7 @@
 		<axis xyz="0 0 1"/>
 		<limit lower="${-170 * M_PI / 180}" upper="${170 * M_PI / 180}" effort="204" velocity="${velocity_scale * 130 * M_PI / 180}" />
+<!--
 		<safety_controller soft_lower_limit="${-168 * M_PI / 180}" soft_upper_limit="${168 * M_PI / 180}" k_position="30" k_velocity="30"/>
+-->
 		<dynamics friction="10.0" damping="1.0"/>
 		<parent link="${name}_4_link"/>
@@ -263,5 +273,7 @@
 		<axis xyz="0 -1 0"/>
 		<limit lower="${-120 * M_PI / 180}" upper="${120 * M_PI / 180}" effort="306" velocity="${velocity_scale * 180 * M_PI / 180}" />
+<!--
 		<safety_controller soft_lower_limit="${-118 * M_PI / 180}" soft_upper_limit="${118 * M_PI / 180}" k_position="30" k_velocity="30"/>
+-->
 		<dynamics friction="10.0" damping="1.0"/>
 		<parent link="${name}_5_link"/>
@@ -293,5 +305,7 @@
 		<axis xyz="0 0 1"/>
 		<limit lower="${-170 * M_PI / 180}" upper="${170 * M_PI / 180}" effort="204" velocity="${velocity_scale * 180 * M_PI / 180}" />
+<!--
 		<safety_controller soft_lower_limit="${-168 * M_PI / 180}" soft_upper_limit="${168 * M_PI / 180}" k_position="30" k_velocity="30"/>
+-->
 		<dynamics friction="10.0" damping="1.0"/>
 		<parent link="${name}_6_link"/>
